Commit message: gazebo

File: hexapod/Hexapod.urdf (robot description, URDF)
Before this commit: robot hexapod, 37 links, 36 joints
Links:
- link Hexapod_Body: geometry collision mesh filename=package://hexapod/meshes/Hexapod_Body.STL; visual mesh filename=package://hexapod/meshes/Hexapod_Body.STL
- link Leg_Five_Foot: geometry collision mesh filename=package://hexapod/meshes/Leg_Five_Foot.STL; visual mesh filename=package://hexapod/meshes/Leg_Five_Foot.STL
- link Leg_Five_Joint_One: geometry collision mesh filename=package://hexapod/meshes/Leg_Five_Joint_One.STL; visual mesh filename=package://hexapod/meshes/Leg_Five_Joint_One.STL
- link Leg_Five_Joint_Two: geometry collision mesh filename=package://hexapod/meshes/Leg_Five_Joint_Two.STL; visual mesh filename=package://hexapod/meshes/Leg_Five_Joint_Two.STL
- link Leg_Five_Motor_One: geometry collision mesh filename=package://hexapod/meshes/Leg_Five_Motor_One.STL; visual mesh filename=package://hexapod/meshes/Leg_Five_Motor_One.STL
- link Leg_Five_Motor_Three: geometry collision mesh filename=package://hexapod/meshes/Leg_Five_Motor_Three.STL; visual mesh filename=package://hexapod/meshes/Leg_Five_Motor_Three.STL
- link Leg_Five_Motor_Two: geometry collision mesh filename=package://hexapod/meshes/Leg_Five_Motor_Two.STL; visual mesh filename=package://hexapod/meshes/Leg_Five_Motor_Two.STL
- link Leg_Four_Foot: geometry collision mesh filename=package://hexapod/meshes/Leg_Four_Foot.STL; visual mesh filename=package://hexapod/meshes/Leg_Four_Foot.STL
- link Leg_Four_Joint_One: geometry collision mesh filename=package://hexapod/meshes/Leg_Four_Joint_One.STL; visual mesh filename=package://hexapod/meshes/Leg_Four_Joint_One.STL
- link Leg_Four_Joint_Two: geometry collision mesh filename=package://hexapod/meshes/Leg_Four_Joint_Two.STL; visual mesh filename=package://hexapod/meshes/Leg_Four_Joint_Two.STL
- link Leg_Four_Motor_One: geometry collision mesh filename=package://hexapod/meshes/Leg_Four_Motor_One.STL; visual mesh filename=package://hexapod/meshes/Leg_Four_Motor_One.STL
- link Leg_Four_Motor_Three: geometry collision mesh filename=package://hexapod/meshes/Leg_Four_Motor_Three.STL; visual mesh filename=package://hexapod/meshes/Leg_Four_Motor_Three.STL
- link Leg_Four_Motor_Two: geometry collision mesh filename=package://hexapod/meshes/Leg_Four_Motor_Two.STL; visual mesh filename=package://hexapod/meshes/Leg_Four_Motor_Two.STL
- link Leg_One_Foot: geometry collision mesh filename=package://hexapod/meshes/Leg_One_Foot.STL; visual mesh filename=package://hexapod/meshes/Leg_One_Foot.STL
- link Leg_One_Joint_One: geometry collision mesh filename=package://hexapod/meshes/Leg_One_Joint_One.STL; visual mesh filename=package://hexapod/meshes/Leg_One_Joint_One.STL
- link Leg_One_Joint_Two: geometry collision mesh filename=package://hexapod/meshes/Leg_One_Joint_Two.STL; visual mesh filename=package://hexapod/meshes/Leg_One_Joint_Two.STL
- link Leg_One_Motor_One: geometry collision mesh filename=package://hexapod/meshes/Leg_One_Motor_One.STL; visual mesh filename=package://hexapod/meshes/Leg_One_Motor_One.STL
- link Leg_One_Motor_Three: geometry collision mesh filename=package://hexapod/meshes/Leg_One_Motor_Three.STL; visual mesh filename=package://hexapod/meshes/Leg_One_Motor_Three.STL
- link Leg_One_Motor_Two: geometry collision mesh filename=package://hexapod/meshes/Leg_One_Motor_Two.STL; visual mesh filename=package://hexapod/meshes/Leg_One_Motor_Two.STL
- link Leg_Six_Foot: geometry collision mesh filename=package://hexapod/meshes/Leg_Six_Foot.STL; visual mesh filename=package://hexapod/meshes/Leg_Six_Foot.STL
- link Leg_Six_Joint_One: geometry collision mesh filename=package://hexapod/meshes/Leg_Six_Joint_One.STL; visual mesh filename=package://hexapod/meshes/Leg_Six_Joint_One.STL
- link Leg_Six_Joint_Two: geometry collision mesh filename=package://hexapod/meshes/Leg_Six_Joint_Two.STL; visual mesh filename=package://hexapod/meshes/Leg_Six_Joint_Two.STL
- link Leg_Six_Motor_One: geometry collision mesh filename=package://hexapod/meshes/Leg_Six_Motor_One.STL; visual mesh filename=package://hexapod/meshes/Leg_Six_Motor_One.STL
- link Leg_Six_Motor_Three: geometry collision mesh filename=package://hexapod/meshes/Leg_Six_Motor_Three.STL; visual mesh filename=package://hexapod/meshes/Leg_Six_Motor_Three.STL
- link Leg_Six_Motor_Two: geometry collision mesh filename=package://hexapod/meshes/Leg_Six_Motor_Two.STL; visual mesh filename=package://hexapod/meshes/Leg_Six_Motor_Two.STL
- link Leg_Three_Foot: geometry collision mesh filename=package://hexapod/meshes/Leg_Three_Foot.STL; visual mesh filename=package://hexapod/meshes/Leg_Three_Foot.STL
- link Leg_Three_Joint_One: geometry collision mesh filename=package://hexapod/meshes/Leg_Three_Joint_One.STL; visual mesh filename=package://hexapod/meshes/Leg_Three_Joint_One.STL
- link Leg_Three_Joint_Two: geometry collision mesh filename=package://hexapod/meshes/Leg_Three_Joint_Two.STL; visual mesh filename=package://hexapod/meshes/Leg_Three_Joint_Two.STL
- link Leg_Three_Motor_One: geometry collision mesh filename=package://hexapod/meshes/Leg_Three_Motor_One.STL; visual mesh filename=package://hexapod/meshes/Leg_Three_Motor_One.STL
- link Leg_Three_Motor_Three: geometry collision mesh filename=package://hexapod/meshes/Leg_Three_Motor_Three.STL; visual mesh filename=package://hexapod/meshes/Leg_Three_Motor_Three.STL
- link Leg_Three_Motor_Two: geometry collision mesh filename=package://hexapod/meshes/Leg_Three_Motor_Two.STL; visual mesh filename=package://hexapod/meshes/Leg_Three_Motor_Two.STL
- link Leg_Two_Foot: geometry collision mesh filename=package://hexapod/meshes/Leg_Two_Foot.STL; visual mesh filename=package://hexapod/meshes/Leg_Two_Foot.STL
- link Leg_Two_Joint_One: geometry collision mesh filename=package://hexapod/meshes/Leg_Two_Joint_One.STL; visual mesh filename=package://hexapod/meshes/Leg_Two_Joint_One.STL
- link Leg_Two_Joint_Two: geometry collision mesh filename=package://hexapod/meshes/Leg_Two_Joint_Two.STL; visual mesh filename=package://hexapod/meshes/Leg_Two_Joint_Two.STL
- link Leg_Two_Motor_One: geometry collision mesh filename=package://hexapod/meshes/Leg_Two_Motor_One.STL; visual mesh filename=package://hexapod/meshes/Leg_Two_Motor_One.STL
- link Leg_Two_Motor_Three: geometry collision mesh filename=package://hexapod/meshes/Leg_Two_Motor_Three.STL; visual mesh filename=package://hexapod/meshes/Leg_Two_Motor_Three.STL
- link Leg_Two_Motor_Two: geometry collision mesh filename=package://hexapod/meshes/Leg_Two_Motor_Two.STL; visual mesh filename=package://hexapod/meshes/Leg_Two_Motor_Two.STL
Joints:
- joint Joint_One_Motor_Five: limit lower=-1.5 upper=1.5 effort=1.5 velocity=6 -> lower=-1.75 upper=1.75 effort=1.5 velocity=6
- joint Joint_One_Motor_Four: limit lower=-1.5 upper=1.5 effort=1.5 velocity=6 -> lower=-1.75 upper=1.75 effort=1.5 velocity=6
- joint Joint_One_Motor_One: limit lower=-1.5 upper=1.5 effort=1.5 velocity=6 -> lower=-1.75 upper=1.75 effort=1.5 velocity=6
- joint Joint_One_Motor_Six: limit lower=-1.5 upper=1.5 effort=1.5 velocity=6 -> lower=-1.75 upper=1.75 effort=1.5 velocity=6
- joint Joint_One_Motor_Three: limit lower=-1.5 upper=1.5 effort=1.5 velocity=6 -> lower=-1.75 upper=1.75 effort=1.5 velocity=6
- joint Joint_One_Motor_Two: limit lower=-1.5 upper=1.5 effort=1.5 velocity=6 -> lower=-1.75 upper=1.75 effort=1.5 velocity=6
- joint Joint_Two_Motor_Five: limit lower=-1.5 upper=1.5 effort=1.5 velocity=6 -> lower=-1.2 upper=1.75 effort=1.5 velocity=6
- joint Joint_Two_Motor_Four: limit lower=-1.5 upper=1.5 effort=1.5 velocity=6 -> lower=-1.2 upper=1.75 effort=1.5 velocity=6
- joint Joint_Two_Motor_One: limit lower=-1.5 upper=1.5 effort=1.5 velocity=6 -> lower=-1.2 upper=1.75 effort=1.5 velocity=6
- joint Joint_Two_Motor_Six: limit lower=-1.5 upper=1.5 effort=1.5 velocity=6 -> lower=-1.2 upper=1.75 effort=1.5 velocity=6
- joint Joint_Two_Motor_Three: limit lower=-1.5 upper=1.5 effort=1.5 velocity=6 -> lower=-1.2 upper=1.75 effort=1.5 velocity=6
- joint Joint_Two_Motor_Two: limit lower=-1.5 upper=1.5 effort=1.5 velocity=6 -> lower=-1.2 upper=1.75 effort=1.5 velocity=6
- joint Motor_One_Joint_Five: limit lower=-1.5 upper=1.5 effort=1.5 velocity=6 -> lower=-0.87 upper=0.87 effort=1.5 velocity=6
- joint Motor_One_Joint_Four: limit lower=-1.5 upper=1.5 effort=1.5 velocity=6 -> lower=-0.87 upper=0.87 effort=1.5 velocity=6
- joint Motor_One_Joint_One: limit lower=-1.5 upper=1.5 effort=1.5 velocity=6 -> lower=-0.87 upper=0.87 effort=1.5 velocity=6
- joint Motor_One_Joint_Six: limit lower=-1.5 upper=1.5 effort=1.5 velocity=6 -> lower=-0.87 upper=0.87 effort=1.5 velocity=6
- joint Motor_One_Joint_Three: limit lower=-1.5 upper=1.5 effort=1.5 velocity=6 -> lower=-0.87 upper=0.87 effort=1.5 velocity=6
- joint Motor_One_Joint_Two: limit lower=-1.5 upper=1.5 effort=1.5 velocity=6 -> lower=-0.87 upper=0.87 effort=1.5 velocity=6

File: hexapod/urdf/Hexapod.urdf (robot description, URDF)
Before this commit: robot Hexapod, 37 links, 36 joints
Links:
- link Hexapod_Body: geometry collision mesh filename=package://hexapod/meshes/Hexapod_Body.STL; visual mesh filename=package://hexapod/meshes/Hexapod_Body.STL
- link Leg_Five_Foot: geometry collision mesh filename=package://hexapod/meshes/Leg_Five_Foot.STL; visual mesh filename=package://hexapod/meshes/Leg_Five_Foot.STL
- link Leg_Five_Joint_One: geometry collision mesh filename=package://hexapod/meshes/Leg_Five_Joint_One.STL; visual mesh filename=package://hexapod/meshes/Leg_Five_Joint_One.STL
- link Leg_Five_Joint_Two: geometry collision mesh filename=package://hexapod/meshes/Leg_Five_Joint_Two.STL; visual mesh filename=package://hexapod/meshes/Leg_Five_Joint_Two.STL
- link Leg_Five_Motor_One: geometry collision mesh filename=package://hexapod/meshes/Leg_Five_Motor_One.STL; visual mesh filename=package://hexapod/meshes/Leg_Five_Motor_One.STL
- link Leg_Five_Motor_Three: geometry collision mesh filename=package://hexapod/meshes/Leg_Five_Motor_Three.STL; visual mesh filename=package://hexapod/meshes/Leg_Five_Motor_Three.STL
- link Leg_Five_Motor_Two: geometry collision mesh filename=package://hexapod/meshes/Leg_Five_Motor_Two.STL; visual mesh filename=package://hexapod/meshes/Leg_Five_Motor_Two.STL
- link Leg_Four_Foot: geometry collision mesh filename=package://hexapod/meshes/Leg_Four_Foot.STL; visual mesh filename=package://hexapod/meshes/Leg_Four_Foot.STL
- link Leg_Four_Joint_One: geometry collision mesh filename=package://hexapod/meshes/Leg_Four_Joint_One.STL; visual mesh filename=package://hexapod/meshes/Leg_Four_Joint_One.STL
- link Leg_Four_Joint_Two: geometry collision mesh filename=package://hexapod/meshes/Leg_Four_Joint_Two.STL; visual mesh filename=package://hexapod/meshes/Leg_Four_Joint_Two.STL
- link Leg_Four_Motor_One: geometry collision mesh filename=package://hexapod/meshes/Leg_Four_Motor_One.STL; visual mesh filename=package://hexapod/meshes/Leg_Four_Motor_One.STL
- link Leg_Four_Motor_Three: geometry collision mesh filename=package://hexapod/meshes/Leg_Four_Motor_Three.STL; visual mesh filename=package://hexapod/meshes/Leg_Four_Motor_Three.STL
- link Leg_Four_Motor_Two: geometry collision mesh filename=package://hexapod/meshes/Leg_Four_Motor_Two.STL; visual mesh filename=package://hexapod/meshes/Leg_Four_Motor_Two.STL
- link Leg_One_Foot: geometry collision mesh filename=package://hexapod/meshes/Leg_One_Foot.STL; visual mesh filename=package://hexapod/meshes/Leg_One_Foot.STL
- link Leg_One_Joint_One: geometry collision mesh filename=package://hexapod/meshes/Leg_One_Joint_One.STL; visual mesh filename=package://hexapod/meshes/Leg_One_Joint_One.STL
- link Leg_One_Joint_Two: geometry collision mesh filename=package://hexapod/meshes/Leg_One_Joint_Two.STL; visual mesh filename=package://hexapod/meshes/Leg_One_Joint_Two.STL
- link Leg_One_Motor_One: geometry collision mesh filename=package://hexapod/meshes/Leg_One_Motor_One.STL; visual mesh filename=package://hexapod/meshes/Leg_One_Motor_One.STL
- link Leg_One_Motor_Three: geometry collision mesh filename=package://hexapod/meshes/Leg_One_Motor_Three.STL; visual mesh filename=package://hexapod/meshes/Leg_One_Motor_Three.STL
- link Leg_One_Motor_Two: geometry collision mesh filename=package://hexapod/meshes/Leg_One_Motor_Two.STL; visual mesh filename=package://hexapod/meshes/Leg_One_Motor_Two.STL
- link Leg_Six_Foot: geometry collision mesh filename=package://hexapod/meshes/Leg_Six_Foot.STL; visual mesh filename=package://hexapod/meshes/Leg_Six_Foot.STL
- link Leg_Six_Joint_One: geometry collision mesh filename=package://hexapod/meshes/Leg_Six_Joint_One.STL; visual mesh filename=package://hexapod/meshes/Leg_Six_Joint_One.STL
- link Leg_Six_Joint_Two: geometry collision mesh filename=package://hexapod/meshes/Leg_Six_Joint_Two.STL; visual mesh filename=package://hexapod/meshes/Leg_Six_Joint_Two.STL
- link Leg_Six_Motor_One: geometry collision mesh filename=package://hexapod/meshes/Leg_Six_Motor_One.STL; visual mesh filename=package://hexapod/meshes/Leg_Six_Motor_One.STL
- link Leg_Six_Motor_Three: geometry collision mesh filename=package://hexapod/meshes/Leg_Six_Motor_Three.STL; visual mesh filename=package://hexapod/meshes/Leg_Six_Motor_Three.STL
- link Leg_Six_Motor_Two: geometry collision mesh filename=package://hexapod/meshes/Leg_Six_Motor_Two.STL; visual mesh filename=package://hexapod/meshes/Leg_Six_Motor_Two.STL
- link Leg_Three_Foot: geometry collision mesh filename=package://hexapod/meshes/Leg_Three_Foot.STL; visual mesh filename=package://hexapod/meshes/Leg_Three_Foot.STL
- link Leg_Three_Joint_One: geometry collision mesh filename=package://hexapod/meshes/Leg_Three_Joint_One.STL; visual mesh filename=package://hexapod/meshes/Leg_Three_Joint_One.STL
- link Leg_Three_Joint_Two: geometry collision mesh filename=package://hexapod/meshes/Leg_Three_Joint_Two.STL; visual mesh filename=package://hexapod/meshes/Leg_Three_Joint_Two.STL
- link Leg_Three_Motor_One: geometry collision mesh filename=package://hexapod/meshes/Leg_Three_Motor_One.STL; visual mesh filename=package://hexapod/meshes/Leg_Three_Motor_One.STL
- link Leg_Three_Motor_Three: geometry collision mesh filename=package://hexapod/meshes/Leg_Three_Motor_Three.STL; visual mesh filename=package://hexapod/meshes/Leg_Three_Motor_Three.STL
- link Leg_Three_Motor_Two: geometry collision mesh filename=package://hexapod/meshes/Leg_Three_Motor_Two.STL; visual mesh filename=package://hexapod/meshes/Leg_Three_Motor_Two.STL
- link Leg_Two_Foot: geometry collision mesh filename=package://hexapod/meshes/Leg_Two_Foot.STL; visual mesh filename=package://hexapod/meshes/Leg_Two_Foot.STL
- link Leg_Two_Joint_One: geometry collision mesh filename=package://hexapod/meshes/Leg_Two_Joint_One.STL; visual mesh filename=package://hexapod/meshes/Leg_Two_Joint_One.STL
- link Leg_Two_Joint_Two: geometry collision mesh filename=package://hexapod/meshes/Leg_Two_Joint_Two.STL; visual mesh filename=package://hexapod/meshes/Leg_Two_Joint_Two.STL
- link Leg_Two_Motor_One: geometry collision mesh filename=package://hexapod/meshes/Leg_Two_Motor_One.STL; visual mesh filename=package://hexapod/meshes/Leg_Two_Motor_One.STL
- link Leg_Two_Motor_Three: geometry collision mesh filename=package://hexapod/meshes/Leg_Two_Motor_Three.STL; visual mesh filename=package://hexapod/meshes/Leg_Two_Motor_Three.STL
- link Leg_Two_Motor_Two: geometry collision mesh filename=package://hexapod/meshes/Leg_Two_Motor_Two.STL; visual mesh filename=package://hexapod/meshes/Leg_Two_Motor_Two.STL
Joints:
- joint Joint_One_Motor_Five: limit lower=-1.75 upper=1.75 effort=1.5 velocity=6 -> lower=-1.5 upper=1.5 effort=1.5 velocity=6
- joint Joint_One_Motor_Four: limit lower=-1.75 upper=1.75 effort=1.5 velocity=6 -> lower=-1.5 upper=1.5 effort=1.5 velocity=6
- joint Joint_One_Motor_One: limit lower=-1.75 upper=1.75 effort=1.5 velocity=6 -> lower=-1.5 upper=1.5 effort=1.5 velocity=6
- joint Joint_One_Motor_Six: limit lower=-1.75 upper=1.75 effort=1.5 velocity=6 -> lower=-1.5 upper=1.5 effort=1.5 velocity=6
- joint Joint_One_Motor_Three: limit lower=-1.75 upper=1.75 effort=1.5 velocity=6 -> lower=-1.5 upper=1.5 effort=1.5 velocity=6
- joint Joint_One_Motor_Two: limit lower=-1.75 upper=1.75 effort=1.5 velocity=6 -> lower=-1.5 upper=1.5 effort=1.5 velocity=6
- joint Joint_Two_Motor_Five: limit lower=-1.2 upper=1.75 effort=1.5 velocity=6 -> lower=-1.5 upper=1.5 effort=1.5 velocity=6
- joint Joint_Two_Motor_Four: limit lower=-1.2 upper=1.75 effort=1.5 velocity=6 -> lower=-1.5 upper=1.5 effort=1.5 velocity=6
- joint Joint_Two_Motor_One: limit lower=-1.2 upper=1.75 effort=1.5 velocity=6 -> lower=-1.5 upper=1.5 effort=1.5 velocity=6
- joint Joint_Two_Motor_Six: limit lower=-1.2 upper=1.75 effort=1.5 velocity=6 -> lower=-1.5 upper=1.5 effort=1.5 velocity=6
- joint Joint_Two_Motor_Three: limit lower=-1.2 upper=1.75 effort=1.5 velocity=6 -> lower=-1.5 upper=1.5 effort=1.5 velocity=6
- joint Joint_Two_Motor_Two: limit lower=-1.2 upper=1.75 effort=1.5 velocity=6 -> lower=-1.5 upper=1.5 effort=1.5 velocity=6
- joint Motor_One_Joint_Five: limit lower=-0.87 upper=0.87 effort=1.5 velocity=6 -> lower=-1.5 upper=1.5 effort=1.5 velocity=6
- joint Motor_One_Joint_Four: limit lower=-0.87 upper=0.87 effort=1.5 velocity=6 -> lower=-1.5 upper=1.5 effort=1.5 velocity=6
- joint Motor_One_Joint_One: limit lower=-0.87 upper=0.87 effort=1.5 velocity=6 -> lower=-1.5 upper=1.5 effort=1.5 velocity=6
- joint Motor_One_Joint_Six: limit lower=-0.87 upper=0.87 effort=1.5 velocity=6 -> lower=-1.5 upper=1.5 effort=1.5 velocity=6
- joint Motor_One_Joint_Three: limit lower=-0.87 upper=0.87 effort=1.5 velocity=6 -> lower=-1.5 upper=1.5 effort=1.5 velocity=6
- joint Motor_One_Joint_Two: limit lower=-0.87 upper=0.87 effort=1.5 velocity=6 -> lower=-1.5 upper=1.5 effort=1.5 velocity=6
